File: DantesqueAutomata_FullSizeBoard/DantesqueAutomata_ADCs.kicad_sch (KiCad schematic)
At the start: 62 parts

Commit message: FullSizeBoard Revision 1 finished
Parts:
- added R21, R23, R25, R27: 5.6kΩ, Resistor_THT:R_Axial_DIN0207_L6.3mm_D2.5mm_P10.16mm_Horizontal, symbol Device:R
- added R22, R24, R26, R28: 2.2kΩ, Resistor_THT:R_Axial_DIN0207_L6.3mm_D2.5mm_P10.16mm_Horizontal, symbol Device:R
- C19, C21, C23, C25, C27, C29, C31, C33, C35, C36, C37, C38, C39, C40, C41, C42: renamed from C?; footprint (none) -> Capacitor_THT:C_Disc_D4.3mm_W1.9mm_P5.00mm
- C20, C22, C24, C26, C28, C30, C32, C34: renamed from C?; footprint (none) -> Capacitor_THT:CP_Radial_D5.0mm_P2.00mm
- R29: renamed from R?; value 130kΩ -> 221Ω; footprint (none) -> Resistor_THT:R_Axial_DIN0207_L6.3mm_D2.5mm_P10.16mm_Horizontal
- R30, R33, R36, R39, R42, R45, R48, R51: renamed from R?; value 120kΩ -> 133kΩ; footprint (none) -> Resistor_THT:R_Axial_DIN0207_L6.3mm_D2.5mm_P10.16mm_Horizontal
- R31, R34, R37, R40, R43, R46, R49, R52: renamed from R?; footprint (none) -> Resistor_THT:R_Axial_DIN0207_L6.3mm_D2.5mm_P10.16mm_Horizontal
- R32, R38, R44, R50: renamed from R?; value 120kΩ -> 221kΩ; footprint (none) -> Resistor_THT:R_Axial_DIN0207_L6.3mm_D2.5mm_P10.16mm_Horizontal
- R35, R41, R47: renamed from R?; value 130kΩ -> 221kΩ; footprint (none) -> Resistor_THT:R_Axial_DIN0207_L6.3mm_D2.5mm_P10.16mm_Horizontal
- U10, U11, U12, U9: renamed from U?; value Opamp_Dual -> LM833
- gave numbers to parts that had none: 2
Connections:
- net GND: now also U9.5 (+), R22.1, R24.1, R26.1, R28.1; no longer U9.6 (-)
- net LIN_1: now also R23.2
- net LIN_2: now also R27.2
- net RIN_1: now also R21.2
- net RIN_2: now also R25.2
- net at C21.1, R32.2, R33.2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: now also U9.6 (-); no longer U9.5 (+)
- new net HD_A_IN1: R21.1, R22.2
- new net HD_A_IN2: R23.1, R24.2
- new net HD_A_IN3: R25.1, R26.2
- new net HD_A_IN4: R27.1, R28.2
Other:
- moved on the sheet: C35, C36, C37, C38, C39, C40, C41, C42, U10C, U11C, U12C, U7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
