File: DantesqueAutomata_FullSizeBoard/DantesqueAutomata_ADCs.kicad_sch (KiCad schematic)
At the start: 62 parts, among them U10 LM833, U11 LM833, U12 LM833, U7 CJMCU-1808, U8 CJMCU-1808, U9 LM833

Commit message: improved pcb design of full size board
Connections:
- net ADC_1 renamed ADC1
- net ADC_2 renamed ADC2
- net ADC_3 renamed ADC3
- net ADC_4 renamed ADC4
- net ADC_5 renamed ADC5
- net ADC_6 renamed ADC6
- net ADC_7 renamed ADC7
- net ADC_8 renamed ADC8
- net BCK_1 renamed BCK1
- net BCK_2 renamed BCK2
- net DIN_1 renamed DIN1
- net DIN_2 renamed DIN2
- net LD_A_IN_1 renamed LD_A_IN1
- net LD_A_IN_2 renamed LD_A_IN2
- net LD_A_IN_3 renamed LD_A_IN3
- net LD_A_IN_4 renamed LD_A_IN4
- net LD_A_IN_5 renamed LD_A_IN5
- net LD_A_IN_6 renamed LD_A_IN6
- net LD_A_IN_7 renamed LD_A_IN7
- net LD_A_IN_8 renamed LD_A_IN8
- net LIN_1 renamed LIN1
- net LIN_2 renamed LIN2
- net MCK_1 renamed MCK1
- net MCK_2 renamed MCK2
- net RIN_1 renamed RIN1
- net RIN_2 renamed RIN2
- net WS_1 renamed WS1
- net WS_2 renamed WS2
