File: DantesqueAutomata_FullSizeBoard/DantesqueAutomata_DACs.kicad_sch (KiCad schematic)
At the start: 42 parts, among them U2 GY-PCM5102, U3 GY-PCM5102, U4 Opamp_Dual, U5 Opamp_Dual, U6 Opamp_Dual, U7 Opamp_Dual

Commit message: FullSizeBoard Revision 1 finished
Parts:
- removed C10, C8: 10µF, symbol Device:C_Polarized
- removed R16: 3.3kΩ, symbol Device:R
- added C11, C9: 10µF, Capacitor_THT:CP_Radial_D5.0mm_P2.00mm, symbol Device:C_Polarized
- added R14, R18: 11kΩ, Resistor_THT:R_Axial_DIN0207_L6.3mm_D2.5mm_P10.16mm_Horizontal, symbol Device:R
- added R17: 80.6kΩ, Resistor_THT:R_Axial_DIN0207_L6.3mm_D2.5mm_P10.16mm_Horizontal, symbol Device:R
- C1, C3: footprint (none) -> Capacitor_THT:CP_Radial_D5.0mm_P2.00mm
- C10: renamed from C9; footprint (none) -> Capacitor_THT:C_Disc_D4.3mm_W1.9mm_P5.00mm
- C12: renamed from C11; footprint (none) -> Capacitor_THT:C_Disc_D4.3mm_W1.9mm_P5.00mm
- C13: renamed from C12; footprint (none) -> Capacitor_THT:C_Disc_D4.3mm_W1.9mm_P5.00mm
- C14: renamed from C13; footprint (none) -> Capacitor_THT:C_Disc_D4.3mm_W1.9mm_P5.00mm
- C15: renamed from C14; footprint (none) -> Capacitor_THT:C_Disc_D4.3mm_W1.9mm_P5.00mm
- C16: renamed from C15; footprint (none) -> Capacitor_THT:C_Disc_D4.3mm_W1.9mm_P5.00mm
- C17: renamed from C16; footprint (none) -> Capacitor_THT:C_Disc_D4.3mm_W1.9mm_P5.00mm
- C18: renamed from C17; footprint (none) -> Capacitor_THT:C_Disc_D4.3mm_W1.9mm_P5.00mm
- C2: footprint (none) -> Capacitor_THT:C_Disc_D4.3mm_W1.9mm_P5.00mm
- C4: renamed from C3; footprint (none) -> Capacitor_THT:C_Disc_D4.3mm_W1.9mm_P5.00mm
- C5: renamed from C4; footprint (none) -> Capacitor_THT:CP_Radial_D5.0mm_P2.00mm
- C6: renamed from C5; footprint (none) -> Capacitor_THT:C_Disc_D4.3mm_W1.9mm_P5.00mm
- C7: renamed from C6; footprint (none) -> Capacitor_THT:CP_Radial_D5.0mm_P2.00mm
- C8: renamed from C7; footprint (none) -> Capacitor_THT:C_Disc_D4.3mm_W1.9mm_P5.00mm
- R1, R10, R11, R12, R2, R3, R4, R5, R6, R7, R8, R9: footprint (none) -> Resistor_THT:R_Axial_DIN0207_L6.3mm_D2.5mm_P10.16mm_Horizontal
- R13: value 3.3kΩ -> 80.6kΩ; footprint (none) -> Resistor_THT:R_Axial_DIN0207_L6.3mm_D2.5mm_P10.16mm_Horizontal
- R15: renamed from R14; value 10kΩ -> 33kΩ; footprint (none) -> Resistor_THT:R_Axial_DIN0207_L6.3mm_D2.5mm_P10.16mm_Horizontal
- R16: renamed from R15; footprint (none) -> Resistor_THT:R_Axial_DIN0207_L6.3mm_D2.5mm_P10.16mm_Horizontal
- R19: renamed from R17; value 10kΩ -> 33kΩ; footprint (none) -> Resistor_THT:R_Axial_DIN0207_L6.3mm_D2.5mm_P10.16mm_Horizontal
- R20: renamed from R18; footprint (none) -> Resistor_THT:R_Axial_DIN0207_L6.3mm_D2.5mm_P10.16mm_Horizontal
- U2, U3: footprint (none) -> Audio_Module:GY-PCM5102
- U4, U5, U6: value Opamp_Dual -> LM833
- U6: renamed from U7; value Opamp_Dual -> LM833
Connections:
- net -12V: now also R13.1, R17.1
- net DAC_1: now also C9.1
- net DAC_2: now also C11.1
- net at C10.1, R13.2, R15.1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: now also R14.2
- net at C12.1, R19.1, U6.6 (-): now also R17.2, R18.2
- net LD_A_OUT1 renamed LD_A_OUT_1
- net LD_A_OUT2 renamed LD_A_OUT_2
- new net: C11.2, R18.1
- new net: C9.2, R14.1

Commit message: improved pcb design of full size board
Connections:
- net BCK_1 renamed BCK1
- net BCK_2 renamed BCK2
- net DAC_1 renamed DAC1
- net DAC_2 renamed DAC2
- net DOUT_1 renamed DOUT1
- net DOUT_2 renamed DOUT2
- net LD_A_OUT_1 renamed LD_A_OUT1
- net LD_A_OUT_2 renamed LD_A_OUT2
- net L_OUT_1 renamed LOUT1
- net L_OUT_2 renamed LOUT2
- net R_OUT_1 renamed ROUT1
- net R_OUT_2 renamed ROUT2
- net WS_1 renamed WS1
- net WS_2 renamed WS2
Changed lines of the file:
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@@
     )
   )
-  (global_label "L_OUT_2" (shape input) (at 203.2 76.2 180) (fields_autoplaced)
+  (global_label "LOUT2" (shape input) (at 203.2 76.2 180) (fields_autoplaced)
     (effects (font (size 1.27 1.27)) (justify right))
-    (property "Intersheet References" "${INTERSHEET_REFS}" (id 0) (at 192.9855 76.1206 0)
+    (property "Intersheet References" "${INTERSHEET_REFS}" (id 0) (at 194.9207 76.1206 0)
       (effects (font (size 1.27 1.27)) (justify right) hide)
     )
   )
-  (global_label "WS_2" (shape input) (at 48.26 80.01 90) (fields_autoplaced)
+  (global_label "WS2" (shape input) (at 48.26 80.01 90) (fields_autoplaced)
     (effects (font (size 1.27 1.27)) (justify left))
-    (property "Intersheet References" "${INTERSHEET_REFS}" (id 0) (at 48.1806 72.7588 90)
+    (property "Intersheet References" "${INTERSHEET_REFS}" (id 0) (at 48.1806 73.7264 90)
       (effects (font (size 1.27 1.27)) (justify left) hide)
     )
   )
-  (global_label "R_OUT_1" (shape input) (at 128.27 41.91 180) (fields_autoplaced)
+  (global_label "ROUT1" (shape input) (at 128.27 41.91 180) (fields_autoplaced)
     (effects (font (size 1.27 1.27)) (justify right))
-    (property "Intersheet References" "${INTERSHEET_REFS}" (id 0) (at 117.8136 41.9894 0)
+    (property "Intersheet References" "${INTERSHEET_REFS}" (id 0) (at 119.7488 41.8306 0)
       (effects (font (size 1.27 1.27)) (justify right) hide)
     )
   )
-  (global_label "DOUT_2" (shape input) (at 50.8 80.01 90) (fields_autoplaced)
+  (global_label "DOUT2" (shape input) (at 50.8 80.01 90) (fields_autoplaced)
     (effects (font (size 1.27 1.27)) (justify left))
-    (property "Intersheet References" "${INTERSHEET_REFS}" (id 0) (at 50.7206 70.5212 90)
+    (property "Intersheet References" "${INTERSHEET_REFS}" (id 0) (at 50.7206 71.4888 90)
       (effects (font (size 1.27 1.27)) (justify left) hide)
     )
   )
-  (global_label "LD_A_OUT_2" (shape input) (at 139.7 177.8 0) (fields_autoplaced)
+  (global_label "LD_A_OUT2" (shape input) (at 139.7 177.8 0) (fields_autoplaced)
     (effects (font (size 1.27 1.27)) (justify left))
-    (property "Intersheet References" "${INTERSHEET_REFS}" (id 0) (at 153.2407 177.7206 0)
+    (property "Intersheet References" "${INTERSHEET_REFS}" (id 0) (at 152.2731 177.7206 0)
       (effects (font (size 1.27 1.27)) (justify left) hide)
     )
@@
     )
   )
-  (global_label "BCK_1" (shape input) (at 53.34 27.94 90) (fields_autoplaced)
+  (global_label "BCK1" (shape input) (at 53.34 27.94 90) (fields_autoplaced)
     (effects (font (size 1.27 1.27)) (justify left))
-    (property "Intersheet References" "${INTERSHEET_REFS}" (id 0) (at 53.2606 19.5398 90)
+    (property "Intersheet References" "${INTERSHEET_REFS}" (id 0) (at 53.2606 20.5074 90)
       (effects (font (size 1.27 1.27)) (justify left) hide)
     )
   )
-  (global_label "R_OUT_2" (shape input) (at 60.96 105.41 0) (fields_autoplaced)
+  (global_label "ROUT2" (shape output) (at 60.96 105.41 0) (fields_autoplaced)
     (effects (font (size 1.27 1.27)) (justify left))
-    (property "Intersheet References" "${INTERSHEET_REFS}" (id 0) (at 71.4164 105.3306 0)
+    (property "Intersheet References" "${INTERSHEET_REFS}" (id 0) (at 69.4812 105.3306 0)
       (effects (font (size 1.27 1.27)) (justify left) hide)
     )
   )
-  (global_label "L_OUT_1" (shape input) (at 60.96 58.42 0) (fields_autoplaced)
+  (global_label "LOUT1" (shape output) (at 60.96 58.42 0) (fields_autoplaced)
     (effects (font (size 1.27 1.27)) (justify left))
-    (property "Intersheet References" "${INTERSHEET_REFS}" (id 0) (at 71.1745 58.4994 0)
+    (property "Intersheet References" "${INTERSHEET_REFS}" (id 0) (at 69.2393 58.3406 0)
       (effects (font (size 1.27 1.27)) (justify left) hide)
     )
   )
-  (global_label "L_OUT_2" (shape input) (at 60.96 110.49 0) (fields_autoplaced)
+  (global_label "LOUT2" (shape output) (at 60.96 110.49 0) (fields_autoplaced)
     (effects (font (size 1.27 1.27)) (justify left))
-    (property "Intersheet References" "${INTERSHEET_REFS}" (id 0) (at 71.1745 110.4106 0)
+    (property "Intersheet References" "${INTERSHEET_REFS}" (id 0) (at 69.2393 110.4106 0)
       (effects (font (size 1.27 1.27)) (justify left) hide)
     )
   )
-  (global_label "R_OUT_1" (shape input) (at 60.96 53.34 0) (fields_autoplaced)
+  (global_label "ROUT1" (shape output) (at 60.96 53.34 0) (fields_autoplaced)
     (effects (font (size 1.27 1.27)) (justify left))
-    (property "Intersheet References" "${INTERSHEET_REFS}" (id 0) (at 71.4164 53.2606 0)
+    (property "Intersheet References" "${INTERSHEET_REFS}" (id 0) (at 69.4812 53.2606 0)
       (effects (font (size 1.27 1.27)) (justify left) hide)
     )
   )
-  (global_label "L_OUT_1" (shape input) (at 128.27 76.2 180) (fields_autoplaced)
+  (global_label "LOUT1" (shape input) (at 128.27 76.2 180) (fields_autoplaced)
     (effects (font (size 1.27 1.27)) (justify right))
-    (property "Intersheet References" "${INTERSHEET_REFS}" (id 0) (at 118.0555 76.1206 0)
+    (property "Intersheet References" "${INTERSHEET_REFS}" (id 0) (at 119.9907 76.1206 0)
       (effects (font (size 1.27 1.27)) (justify right) hide)
     )
   )
-  (global_label "R_OUT_2" (shape input) (at 203.2 41.91 180) (fields_autoplaced)
+  (global_label "ROUT2" (shape input) (at 203.2 41.91 180) (fields_autoplaced)
     (effects (font (size 1.27 1.27)) (justify right))
-    (property "Intersheet References" "${INTERSHEET_REFS}" (id 0) (at 192.7436 41.8306 0)
+    (property "Intersheet References" "${INTERSHEET_REFS}" (id 0) (at 194.6788 41.8306 0)
       (effects (font (size 1.27 1.27)) (justify right) hide)
     )
@@
     )
   )
-  (global_label "DAC_1" (shape input) (at 92.71 140.97 180) (fields_autoplaced)
+  (global_label "DAC1" (shape input) (at 92.71 140.97 180) (fields_autoplaced)
     (effects (font (size 1.27 1.27)) (justify right))
-    (property "Intersheet References" "${INTERSHEET_REFS}" (id 0) (at 84.4912 140.8906 0)
+    (property "Intersheet References" "${INTERSHEET_REFS}" (id 0) (at 85.4588 140.8906 0)
       (effects (font (size 1.27 1.27)) (justify right) hide)
     )
   )
-  (global_label "DOUT_1" (shape input) (at 50.8 27.94 90) (fields_autoplaced)
+  (global_label "DOUT1" (shape input) (at 50.8 27.94 90) (fields_autoplaced)
     (effects (font (size 1.27 1.27)) (justify left))
-    (property "Intersheet References" "${INTERSHEET_REFS}" (id 0) (at 50.7206 18.4512 90)
+    (property "Intersheet References" "${INTERSHEET_REFS}" (id 0) (at 50.7206 19.4188 90)
       (effects (font (size 1.27 1.27)) (justify left) hide)
     )
   )
-  (global_label "BCK_2" (shape input) (at 53.34 80.01 90) (fields_autoplaced)
+  (global_label "BCK2" (shape input) (at 53.34 80.01 90) (fields_autoplaced)
     (effects (font (size 1.27 1.27)) (justify left))
-    (property "Intersheet References" "${INTERSHEET_REFS}" (id 0) (at 53.2606 71.6098 90)
+    (property "Intersheet References" "${INTERSHEET_REFS}" (id 0) (at 53.2606 72.5774 90)
       (effects (font (size 1.27 1.27)) (justify left) hide)
     )
   )
-  (global_label "DAC_2" (shape input) (at 92.71 175.26 180) (fields_autoplaced)
+  (global_label "DAC2" (shape input) (at 92.71 175.26 180) (fields_autoplaced)
     (effects (font (size 1.27 1.27)) (justify right))
-    (property "Intersheet References" "${INTERSHEET_REFS}" (id 0) (at 84.4912 175.1806 0)
+    (property "Intersheet References" "${INTERSHEET_REFS}" (id 0) (at 85.4588 175.1806 0)
       (effects (font (size 1.27 1.27)) (justify right) hide)
     )
   )
-  (global_label "WS_1" (shape input) (at 48.26 27.94 90) (fields_autoplaced)
+  (global_label "WS1" (shape input) (at 48.26 27.94 90) (fields_autoplaced)
     (effects (font (size 1.27 1.27)) (justify left))
-    (property "Intersheet References" "${INTERSHEET_REFS}" (id 0) (at 48.1806 20.6888 90)
+    (property "Intersheet References" "${INTERSHEET_REFS}" (id 0) (at 48.1806 21.6564 90)
       (effects (font (size 1.27 1.27)) (justify left) hide)
     )
   )
-  (global_label "LD_A_OUT_1" (shape input) (at 139.7 143.51 0) (fields_autoplaced)
+  (global_label "LD_A_OUT1" (shape input) (at 139.7 143.51 0) (fields_autoplaced)
     (effects (font (size 1.27 1.27)) (justify left))
-    (property "Intersheet References" "${INTERSHEET_REFS}" (id 0) (at 153.2407 143.4306 0)
+    (property "Intersheet References" "${INTERSHEET_REFS}" (id 0) (at 152.2731 143.4306 0)
       (effects (font (size 1.27 1.27)) (justify left) hide)
     )
